File: r2021-02/hubbish-rev2.kicad_sch (KiCad schematic)
At the start: 4 parts

Commit message: overhaul, push silk, complete "again"
Parts:
- added TP1, TP2, TP3: TestPoint, et-parts:TestPoint_Plated_Hole_0.6_D0.8mm, symbol Connector:TestPoint
Connections:
- new net +3V3: TP2.1
- new net +5V: TP1.1
- new net GND: TP3.1

Commit message: r2: push more, switch to m3 mounting, more silk
added a chicken jumper to connect vbus and 5v...
Parts:
- H1, H2, H3, H4: footprint MountingHole:MountingHole_2.7mm_M2.5 -> MountingHole:MountingHole_3.2mm_M3
