File: r2021-02/power_input.kicad_sch (KiCad schematic)
At the start: 28 parts, among them J8 Conn_01x06, Q1 Si4435, U18 SiC437AED, U19 SE5120ST33

Commit message: BOM revisions for a rev3
Probably not going to bother even assembling rev2 pcbs.  Was missing
parts, found other things that were a little non-ideal.

Decided to start revising towards making it assembleable by JLC, so
using super cheap parts from their basic line where possible, and
minimizing bom items.
Parts:
- removed C40, C42: 100uF, Capacitor_SMD:CP_Elec_5x5.4, symbol Device:C_Polarized_Small
- removed C43: 22uF/6.3V, Capacitor_SMD:C_0805_2012Metric, symbol Device:C_Small
- added C36, C37: 10uF/30+, Capacitor_SMD:C_1206_3216Metric, symbol Device:C_Small
- added C42: 100nF, Capacitor_SMD:C_0603_1608Metric, symbol Device:C_Small
- added C44, C46, C48: 10uF-up?, Capacitor_SMD:C_0603_1608Metric, symbol Device:C_Small
- C34, C35: value 22uF/30V+ -> 10uF/30+; footprint Capacitor_SMD:C_0805_2012Metric -> Capacitor_SMD:C_1206_3216Metric; MPN (none) -> CL31A106KBHNNNE; jlc-basic (none) -> 1; lcsc# (none) -> C13585
- C38: renamed from C36; value .1uF -> 100nF/30+; MPN (none) -> CC0603KRX7R9BB104; jlc-basic (none) -> 1; lcsc# (none) -> C14663
- C39: renamed from C37; MPN (none) -> CL10A105KB8NNNC; jlc-basic (none) -> 1; lcsc# (none) -> C15849
- C40: renamed from C38; value 4.7uF -> 1uF; MPN (none) -> CL10A105KB8NNNC; jlc-basic (none) -> 1; lcsc# (none) -> C15849
- C41: renamed from C39; value .1uF -> 100nF; MPN (none) -> CC0603KRX7R9BB104; jlc-basic (none) -> 1; lcsc# (none) -> C14663
- C43: renamed from C41; footprint Capacitor_SMD:C_0805_2012Metric -> Capacitor_SMD:C_0603_1608Metric; MPN (none) -> CL10A106KP8NNNC; jlc-basic (none) -> 1; lcsc# (none) -> C19702
- C45: value 22uF/6.3V -> 10uF-up?; footprint Capacitor_SMD:C_0805_2012Metric -> Capacitor_SMD:C_0603_1608Metric; MPN (none) -> CL10A106KP8NNNC; jlc-basic (none) -> 1; lcsc# (none) -> C19702
- C47: renamed from C44; footprint Capacitor_SMD:C_0805_2012Metric -> Capacitor_SMD:C_0603_1608Metric; MPN (none) -> CL10A106KP8NNNC; jlc-basic (none) -> 1; lcsc# (none) -> C19702
- R24: renamed from R23; MPN (none) -> 0603WAF1002T5E; jlc-basic (none) -> 1; lcsc# (none) -> C25804
- R26: renamed from R25; MPN (none) -> 0603WAF1003T5E; jlc-basic (none) -> 1; lcsc# (none) -> C25803
- R28: renamed from R27; value 499k -> 510k; MPN (none) -> 0603WAF5103T5E; jlc-basic (none) -> 1; lcsc# (none) -> C23192
- R29: renamed from R28; value 2.2 -> 0; MPN (none) -> 0603WAF0000T5E; jlc-basic (none) -> 1; lcsc# (none) -> C21189
- R30: renamed from R29; value 22k -> 75k; MPN (none) -> 0603WAF7502T5E; jlc-basic (none) -> 1; lcsc# (none) -> C23242
- R31: renamed from R30; value 3k -> 10k; MPN (none) -> 0603WAF1002T5E; jlc-basic (none) -> 1; lcsc# (none) -> C25804
- renumbered R24 to R25, R26 to R27
Connections:
- net +5V: now also C42.1, C44.1, C46.1, C48.1
- net +VDC: now also C36.1, C37.1
- net GND: now also C36.2, C37.2, C42.2, C44.2, C46.2, C48.2
Other:
- note added: "73.2k=> 4.93 out 75k => 5.1 out... better... I think."
- note added: "DS says COUT = 47 μF x 7 (329uF), CIN = 10 μF x 6, "unless otherwise noted" (for specs!) eval board hsa 3x22uF+100nF on in and 2x22uF+100nF on output ds has 2x22uF+100nf on input, plus 4x47uF on output?! perhaps, 4x10uF? for 4x10uF for 30V+ is"
- note added: "Switch to Sic402, it's available for assembly at jlc and is also available on mouser"
- note added: "ds says 2.2 and 4.7, diff places evb has 1u 1u is _great_ for bom"
- note added: "evb has 0 here for phase!"
- note added: "min 10uF using 22uF for BOM optimization"
