File: r2022-10/r2022-10.kicad_sch (KiCad schematic)
At the start: 7 parts

Commit message: rev3: overhaul nearly all parts to be from jlc pcba
Only the inductor left.  I've marked a few through hole parts as DNP, as
I can solder them by hand, and already have the parts in stock.  But
everything else goes to JLC for assembly, with every attempt made to
stick to only basic parts, or shared parts.  Beyond that, price and
stocking!
Parts:
- H1, H2, H3, H4, TP1, TP2, TP3: DNP (none) -> 1
