File: r2022-10/upstream-config-leds.kicad_sch (KiCad schematic)
At the start: 60 parts, among them J1 Conn_01x03_Male, J2 USB_A male UP, J3 USB_B_Micro (up), U1 2k i2c eeprom, U2 NUP4202, U3 USB2517, Y1 24MHz

Commit message: rev3: overhaul nearly all parts to be from jlc pcba
Only the inductor left.  I've marked a few through hole parts as DNP, as
I can solder them by hand, and already have the parts in stock.  But
everything else goes to JLC for assembly, with every attempt made to
stick to only basic parts, or shared parts.  Beyond that, price and
stocking!
Parts:
- D1: footprint LED_SMD:LED_0603_1608Metric -> LED_SMD:LED_0805_2012Metric; MPN (none) -> NCD0805R1; jlc-basic (none) -> 1; lcsc# (none) -> C84256
- D10, D4, D5, D6, D7, D8, D9: value LTST-C295KGKRKT -> LTST-C195KGJRKT; footprint LED_SMD:LED_LiteOn_LTST-C295K -> LED_Dual:T1615_LiteOn_LTST_C195x; MPN (none) -> LTST-C195KGJRKT; jlc-basic (none) -> 0; lcsc# (none) -> C125104
- D2: footprint LED_SMD:LED_0603_1608Metric -> LED_SMD:LED_0805_2012Metric; DNP (none) -> 1; MPN (none) -> NCD0805R1; jlc-basic (none) -> 1; lcsc# (none) -> C84256
- D3: MPN (none) -> SM4007PL; jlc-basic (none) -> 1; lcsc# (none) -> C64898
- J1, J2, JP1, JP2, R3, R6, R8: DNP (none) -> 1
- J3: jlc-basic (none) -> 0; lcsc# (none) -> C319164
- Y1: MPN CF4024M00012T8188046 -> X322524MOB4SI; lcsc# C709021 -> C70590
Other:
- note added: "This current part is discontinued look for a replacement, should be easy enough"

Commit message: r3: add power good led, add auto switch 5v sources
copied from nanopi usb sections.

still need to adjust the spacing of the leds, and decide on ordering,
with or without eeprom permanently.
Parts:
- added Q2, Q4: S8550, Package_TO_SOT_SMD:SOT-23, symbol Device:Q_PNP_BEC
- added Q3: AO3401A, Package_TO_SOT_SMD:SOT-23, symbol Transistor_FET:AO3401A
- added R15, R16: 10k, Resistor_SMD:R_0603_1608Metric, symbol Device:R_Small
- renumbered R14 to R13, R15 to R14, R16 to R17, R17 to R18, R18 to R19, R19 to R20, R20 to R21, R21 to R22, R22 to R32, R23 to R33
Connections:
- net +5V: now also Q3.2 (S), Q4.2 (E)
- net GND: now also R15.2, R16.2
- net VBUS_UP: now also Q2.2 (E), Q3.3 (D)
- new net: Q2.1 (B), Q2.3 (C), Q4.1 (B), R15.1
- new net: Q3.1 (G), Q4.3 (C), R16.1
Other:
- note added: "Copied from NanoPi boards"

Commit message: r3: save all laast edits too
Parts:
- C1, C10, C11, C12, C14, C15, C16, C18, C19, C2, C3, C8: lcsc# C14663 -> C14663
Changed lines of the file:
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@@
       (effects (font (size 1.27 1.27)) hide)
     )
-    (property "lcsc#" " C14663 " (id 5) (at 256.54 35.56 0)
+    (property "lcsc#" "C14663" (id 5) (at 256.54 35.56 0)
       (effects (font (size 1.27 1.27)) hide)
     )
@@
       (effects (font (size 1.27 1.27)) hide)
     )
-    (property "lcsc#" " C14663 " (id 5) (at 226.06 35.56 0)
+    (property "lcsc#" "C14663" (id 5) (at 226.06 35.56 0)
       (effects (font (size 1.27 1.27)) hide)
     )
@@
       (effects (font (size 1.27 1.27)) hide)
     )
-    (property "lcsc#" " C14663 " (id 5) (at 233.68 35.56 0)
+    (property "lcsc#" "C14663" (id 5) (at 233.68 35.56 0)
       (effects (font (size 1.27 1.27)) hide)
     )
@@
       (effects (font (size 1.27 1.27)) hide)
     )
-    (property "lcsc#" " C14663 " (id 5) (at 241.3 35.56 0)
+    (property "lcsc#" "C14663" (id 5) (at 241.3 35.56 0)
       (effects (font (size 1.27 1.27)) hide)
     )
@@
       (effects (font (size 1.27 1.27)) hide)
     )
-    (property "lcsc#" " C14663 " (id 5) (at 248.92 35.56 0)
+    (property "lcsc#" "C14663" (id 5) (at 248.92 35.56 0)
       (effects (font (size 1.27 1.27)) hide)
     )
@@
       (effects (font (size 1.27 1.27)) hide)
     )
-    (property "lcsc#" " C14663 " (id 5) (at 254 121.92 0)
+    (property "lcsc#" "C14663" (id 5) (at 254 121.92 0)
       (effects (font (size 1.27 1.27)) hide)
     )
@@
       (effects (font (size 1.27 1.27)) hide)
     )
-    (property "lcsc#" " C14663 " (id 5) (at 269.24 121.92 0)
+    (property "lcsc#" "C14663" (id 5) (at 269.24 121.92 0)
       (effects (font (size 1.27 1.27)) hide)
     )
@@
       (effects (font (size 1.27 1.27)) hide)
     )
-    (property "lcsc#" " C14663 " (id 5) (at 160.02 129.54 0)
+    (property "lcsc#" "C14663" (id 5) (at 160.02 129.54 0)
       (effects (font (size 1.27 1.27)) hide)
     )
@@
       (effects (font (size 1.27 1.27)) hide)
     )
-    (property "lcsc#" " C14663 " (id 5) (at 50.8 152.4 0)
+    (property "lcsc#" "C14663" (id 5) (at 50.8 152.4 0)
       (effects (font (size 1.27 1.27)) hide)
     )
@@
       (effects (font (size 1.27 1.27)) hide)
     )
-    (property "lcsc#" " C14663 " (id 5) (at 198.12 35.56 0)
+    (property "lcsc#" "C14663" (id 5) (at 198.12 35.56 0)
       (effects (font (size 1.27 1.27)) hide)
     )
@@
       (effects (font (size 1.27 1.27)) hide)
     )
-    (property "lcsc#" " C14663 " (id 5) (at 264.16 35.56 0)
+    (property "lcsc#" "C14663" (id 5) (at 264.16 35.56 0)
       (effects (font (size 1.27 1.27)) hide)
     )
@@
       (effects (font (size 1.27 1.27)) hide)
     )
-    (property "lcsc#" " C14663 " (id 5) (at 71.12 68.58 0)
-      (effects (font (size 1.27 1.27)) hide)
-    )
+    (property "lcsc#" "C14663" (id 5) (at 71.12 68.58 0)
+      (effects (font (size 1.27 1.27)) hide)
+    )

Commit message: rev3-2022-10: add fixme text on errors
Other:
- note added: "Copied from NanoPi boards (But badly, these should have been a matched pair eg bcm856bs (as they used) or mpn:BCM857BS-7-F lcsc: C105896"
- note added: "FIXME - "local power" can't just be 3v3. that's always there, whether 3v3 came from vbus or vext!"
- note removed: "Copied from NanoPi boards"
Changed lines of the file:
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@@
+    (effects (font (size 1.27 1.27)) (justify left bottom))
+  )
+  (text "FIXME - \"local power\" can't just be 3v3.\nthat's always there, whether 3v3 came\nfrom vbus or vext!"
+    (at 137.16 33.02 0)
     (effects (font (size 1.27 1.27)) (justify left bottom))
   )
@@
     (effects (font (size 0.9906 0.9906)) (justify left bottom))
   )
-  (text "Copied from NanoPi boards" (at 228.6 251.46 0)
+  (text "Copied from NanoPi boards\n(But badly, these should have been a matched pair\neg bcm856bs (as they used) or \nmpn:BCM857BS-7-F lcsc: C105896"
+    (at 218.44 261.62 0)
     (effects (font (size 1.27 1.27)) (justify left bottom))
   )
